Commit message: imu added and interfaced '

File: robot_navigation/robot_nav_description/models/diff_drive/model.urdf (robot description, URDF)
Before this commit: robot diff_drive, 6 links, 5 joints
Links:
- added link imu_link, mass 0.01
- link caster: mass 0.5 -> 2.0
Joints:
- added joint imu_joint: type fixed, parent chassis, child imu_link, origin xyz=0 0 0.2 rpy=0 0 0
